Commit message: modify wal

File: sim/field.urdf (robot description, URDF)
Before this commit: robot large_cube, 14 links, 12 joints
Links:
- removed link left_side_net
- link left_side_wall_1: geometry collision box size=0.01 0.1 0.54; visual box size=0.01 0.1 0.54
- link left_side_wall_2: geometry collision box size=0.01 0.35 0.54; visual box size=0.01 0.35 0.54
- link left_side_wall_3: geometry collision box size=0.01 0.35 0.54; visual box size=0.01 0.35 0.54
- link left_side_wall_4: geometry collision box size=0.01 0.1 0.54; visual box size=0.01 0.1 0.54
Joints:
- joint left_side_wall_1_fixed_joint: origin xyz=-0.1325 0.05 0.27 rpy=0 0 0 -> xyz=-0.005 0.05 0.27 rpy=0 0 0
- joint left_side_wall_2_fixed_joint: origin xyz=-0.1325 0.575 0.27 rpy=0 0 0 -> xyz=-0.005 0.575 0.27 rpy=0 0 0
- joint left_side_wall_3_fixed_joint: origin xyz=-0.1325 1.225 0.27 rpy=0 0 0 -> xyz=-0.005 1.225 0.27 rpy=0 0 0
- joint left_side_wall_4_fixed_joint: origin xyz=-0.1325 1.75 0.27 rpy=0 0 0 -> xyz=-0.005 1.75 0.27 rpy=0 0 0

Commit message: add blue post

File: sim/field.urdf (robot description, URDF)
Before this commit: robot large_cube, 13 links, 12 joints
Links:
- added link left_side_blue_post_1, mass 1; collision box size=0.255 0.1 0.54; visual box size=0.255 0.1 0.54
- added link left_side_blue_post_2, mass 1; collision box size=0.255 0.1 0.54; visual box size=0.255 0.1 0.54
- added link left_side_blue_post_3, mass 1; collision box size=0.01 0.5 0.84; visual box size=0.01 0.5 0.84
Joints:
- added joint left_side_blue_post_1_fixed_joint: type fixed, parent main_field, child left_side_blue_post_1, origin xyz=-0.1375 0.05 0.27 rpy=0 0 0
- added joint left_side_blue_post_2_fixed_joint: type fixed, parent main_field, child left_side_blue_post_2, origin xyz=-0.1375 0.45 0.27 rpy=0 0 0
- added joint left_side_blue_post_3_fixed_joint: type fixed, parent main_field, child left_side_blue_post_3, origin xyz=-0.270 0.25 0.42 rpy=0 0 0

Commit message: add yellow post

File: sim/field.urdf (robot description, URDF)
Before this commit: robot large_cube, 16 links, 15 joints
Links:
- added link left_side_yellow_post_1, mass 1; collision box size=0.255 0.1 0.54; visual box size=0.255 0.1 0.54
- added link left_side_yellow_post_2, mass 1; collision box size=0.255 0.1 0.54; visual box size=0.255 0.1 0.54
- added link left_side_yellow_post_3, mass 1; collision box size=0.01 0.5 0.84; visual box size=0.01 0.5 0.84
Joints:
- added joint left_side_yellow_post_1_fixed_joint: type fixed, parent main_field, child left_side_yellow_post_1, origin xyz=-0.1375 0.7 0.27 rpy=0 0 0
- added joint left_side_yellow_post_2_fixed_joint: type fixed, parent main_field, child left_side_yellow_post_2, origin xyz=-0.1375 1.1 0.27 rpy=0 0 0
- added joint left_side_yellow_post_3_fixed_joint: type fixed, parent main_field, child left_side_yellow_post_3, origin xyz=-0.270 0.9 0.42 rpy=0 0 0

Commit message: fix color blue to red

File: sim/field.urdf (robot description, URDF)
Before this commit: robot large_cube, 19 links, 18 joints
Links:
- removed link left_side_blue_post_1
- removed link left_side_blue_post_2
- removed link left_side_blue_post_3
- added link left_side_red_post_1, mass 1; collision box size=0.255 0.1 0.54; visual box size=0.255 0.1 0.54
- added link left_side_red_post_2, mass 1; collision box size=0.255 0.1 0.54; visual box size=0.255 0.1 0.54
- added link left_side_red_post_3, mass 1; collision box size=0.01 0.5 0.84; visual box size=0.01 0.5 0.84
Joints:
- removed joint left_side_blue_post_1_fixed_joint
- removed joint left_side_blue_post_2_fixed_joint
- removed joint left_side_blue_post_3_fixed_joint
- added joint left_side_red_post_1_fixed_joint: type fixed, parent main_field, child left_side_red_post_1, origin xyz=-0.1375 0.05 0.27 rpy=0 0 0
- added joint left_side_red_post_2_fixed_joint: type fixed, parent main_field, child left_side_red_post_2, origin xyz=-0.1375 0.45 0.27 rpy=0 0 0
- added joint left_side_red_post_3_fixed_joint: type fixed, parent main_field, child left_side_red_post_3, origin xyz=-0.270 0.25 0.42 rpy=0 0 0

Commit message: add blue post

File: sim/field.urdf (robot description, URDF)
Before this commit: robot large_cube, 19 links, 18 joints
Links:
- added link left_side_blue_post_1, mass 1; collision box size=0.255 0.1 0.54; visual box size=0.255 0.1 0.54
- added link left_side_blue_post_2, mass 1; collision box size=0.255 0.1 0.54; visual box size=0.255 0.1 0.54
- added link left_side_blue_post_3, mass 1; collision box size=0.01 0.5 0.84; visual box size=0.01 0.5 0.84
Joints:
- added joint left_side_blue_post_1_fixed_joint: type fixed, parent main_field, child left_side_blue_post_1, origin xyz=-0.1375 1.35 0.27 rpy=0 0 0
- added joint left_side_blue_post_2_fixed_joint: type fixed, parent main_field, child left_side_blue_post_2, origin xyz=-0.1375 1.75 0.27 rpy=0 0 0
- added joint left_side_blue_post_3_fixed_joint: type fixed, parent main_field, child left_side_blue_post_3, origin xyz=-0.270 1.55 0.42 rpy=0 0 0

Commit message: fix left post hight

File: sim/field.urdf (robot description, URDF)
Before this commit: robot large_cube, 22 links, 21 joints
Links:
- link left_side_blue_post_1: geometry collision box size=0.255 0.1 0.5; visual box size=0.255 0.1 0.5
- link left_side_blue_post_2: geometry collision box size=0.255 0.1 0.5; visual box size=0.255 0.1 0.5
- link left_side_blue_post_3: geometry collision box size=0.01 0.5 0.8; visual box size=0.01 0.5 0.8
- link left_side_red_post_1: geometry collision box size=0.255 0.1 0.5; visual box size=0.255 0.1 0.5
- link left_side_red_post_2: geometry collision box size=0.255 0.1 0.5; visual box size=0.255 0.1 0.5
- link left_side_red_post_3: geometry collision box size=0.01 0.5 0.8; visual box size=0.01 0.5 0.8
- link left_side_yellow_post_1: geometry collision box size=0.255 0.1 0.5; visual box size=0.255 0.1 0.5
- link left_side_yellow_post_2: geometry collision box size=0.255 0.1 0.5; visual box size=0.255 0.1 0.5
- link left_side_yellow_post_3: geometry collision box size=0.01 0.5 0.8; visual box size=0.01 0.5 0.8
Joints:
- joint left_side_blue_post_1_fixed_joint: origin xyz=-0.1375 1.35 0.27 rpy=0 0 0 -> xyz=-0.1375 1.35 0.25 rpy=0 0 0
- joint left_side_blue_post_2_fixed_joint: origin xyz=-0.1375 1.75 0.27 rpy=0 0 0 -> xyz=-0.1375 1.75 0.25 rpy=0 0 0
- joint left_side_blue_post_3_fixed_joint: origin xyz=-0.270 1.55 0.42 rpy=0 0 0 -> xyz=-0.270 1.55 0.4 rpy=0 0 0
- joint left_side_red_post_1_fixed_joint: origin xyz=-0.1375 0.05 0.27 rpy=0 0 0 -> xyz=-0.1375 0.05 0.25 rpy=0 0 0
- joint left_side_red_post_2_fixed_joint: origin xyz=-0.1375 0.45 0.27 rpy=0 0 0 -> xyz=-0.1375 0.45 0.25 rpy=0 0 0
- joint left_side_red_post_3_fixed_joint: origin xyz=-0.270 0.25 0.42 rpy=0 0 0 -> xyz=-0.270 0.25 0.4 rpy=0 0 0
- joint left_side_yellow_post_1_fixed_joint: origin xyz=-0.1375 0.7 0.27 rpy=0 0 0 -> xyz=-0.1375 0.7 0.25 rpy=0 0 0
- joint left_side_yellow_post_2_fixed_joint: origin xyz=-0.1375 1.1 0.27 rpy=0 0 0 -> xyz=-0.1375 1.1 0.25 rpy=0 0 0
- joint left_side_yellow_post_3_fixed_joint: origin xyz=-0.270 0.9 0.42 rpy=0 0 0 -> xyz=-0.270 0.9 0.4 rpy=0 0 0

Commit message: base down to the ground

File: sim/field.urdf (robot description, URDF)
Before this commit: robot large_cube, 22 links, 21 joints
Links:
- removed link left_side_blue_post_1
- removed link left_side_blue_post_2
- removed link left_side_red_post_1
- removed link left_side_red_post_2
- removed link left_side_yellow_post_1
- removed link left_side_yellow_post_2
- removed link main_field
- removed link start_area
- added link base_point, mass 1; collision box size=0.001 0.001 0.001; visual box size=0.001 0.001 0.001
- link bottom_side_wall: geometry collision box size=1.3 0.01 0.04; visual box size=1.3 0.01 0.04
- link left_side_blue_post_3: geometry collision box size=0.01 0.5 0.3; visual box size=0.01 0.5 0.3
- link left_side_red_post_3: geometry collision box size=0.01 0.5 0.3; visual box size=0.01 0.5 0.3
- link left_side_wall_1: geometry collision box size=0.01 0.1 0.04; visual box size=0.01 0.1 0.04
- link left_side_wall_2: geometry collision box size=0.01 0.35 0.04; visual box size=0.01 0.35 0.04
- link left_side_wall_3: geometry collision box size=0.01 0.35 0.04; visual box size=0.01 0.35 0.04
- link left_side_wall_4: geometry collision box size=0.01 0.1 0.04; visual box size=0.01 0.1 0.04
- link left_side_yellow_post_3: geometry collision box size=0.01 0.5 0.3; visual box size=0.01 0.5 0.3
- link right_side_wall: geometry collision box size=0.01 1.8 0.04; visual box size=0.01 1.8 0.04
- link start_bottom_side_wall: geometry collision box size=0.5 0.01 0.04; visual box size=0.5 0.01 0.04
- link start_left_side_wall: geometry collision box size=0.01 0.5 0.04; visual box size=0.01 0.5 0.04
- link start_right_side_wall: geometry collision box size=0.01 0.5 0.04; visual box size=0.01 0.5 0.04
- link top_side_wall: geometry collision box size=1.8 0.01 0.04; visual box size=1.8 0.01 0.04
Joints:
- removed joint left_side_blue_post_1_fixed_joint
- removed joint left_side_blue_post_2_fixed_joint
- removed joint left_side_red_post_1_fixed_joint
- removed joint left_side_red_post_2_fixed_joint
- removed joint left_side_yellow_post_1_fixed_joint
- removed joint left_side_yellow_post_2_fixed_joint
- removed joint small_cube_fixed_joint
- joint bottom_side_wall_fixed_joint: origin xyz=1.15 -0.005 0.27 rpy=0 0 0 -> xyz=1.15 -0.005 0.02 rpy=0 0 0; parent main_field -> base_point
- joint center_island_fixed_joint: origin xyz=0.74 0.85 0.52 rpy=0 0 0 -> xyz=0.9 0.9 0.02 rpy=0 0 0; parent main_field -> base_point
- joint left_side_blue_post_3_fixed_joint: origin xyz=-0.270 1.55 0.4 rpy=0 0 0 -> xyz=-0.270 1.55 0.15 rpy=0 0 0; parent main_field -> base_point
- joint left_side_red_post_3_fixed_joint: origin xyz=-0.270 0.25 0.4 rpy=0 0 0 -> xyz=-0.270 0.25 0.15 rpy=0 0 0; parent main_field -> base_point
- joint left_side_wall_1_fixed_joint: origin xyz=-0.005 0.05 0.27 rpy=0 0 0 -> xyz=-0.005 0.05 0.02 rpy=0 0 0; parent main_field -> base_point
- joint left_side_wall_2_fixed_joint: origin xyz=-0.005 0.575 0.27 rpy=0 0 0 -> xyz=-0.005 0.575 0.02 rpy=0 0 0; parent main_field -> base_point
- joint left_side_wall_3_fixed_joint: origin xyz=-0.005 1.225 0.27 rpy=0 0 0 -> xyz=-0.005 1.225 0.02 rpy=0 0 0; parent main_field -> base_point
- joint left_side_wall_4_fixed_joint: origin xyz=-0.005 1.75 0.27 rpy=0 0 0 -> xyz=-0.005 1.75 0.02 rpy=0 0 0; parent main_field -> base_point
- joint left_side_yellow_post_3_fixed_joint: origin xyz=-0.270 0.9 0.4 rpy=0 0 0 -> xyz=-0.270 0.9 0.15 rpy=0 0 0; parent main_field -> base_point
- joint right_side_wall_fixed_joint: origin xyz=1.805 0.9 0.27 rpy=0 0 0 -> xyz=1.805 0.9 0.02 rpy=0 0 0; parent main_field -> base_point
- joint start_bottom_side_wall_fixed_joint: origin xyz=0.25 -0.505 0.27 rpy=0 0 0 -> xyz=0.25 -0.505 0.02 rpy=0 0 0; parent main_field -> base_point
- joint start_left_side_wall_fixed_joint: origin xyz=-0.005 -0.25 0.27 rpy=0 0 0 -> xyz=-0.005 -0.25 0.02 rpy=0 0 0; parent main_field -> base_point
- joint start_right_side_wall_fixed_joint: origin xyz=0.505 -0.25 0.27 rpy=0 0 0 -> xyz=0.505 -0.25 0.02 rpy=0 0 0; parent main_field -> base_point
- joint top_side_wall_fixed_joint: origin xyz=0.9 1.805 0.27 rpy=0 0 0 -> xyz=0.9 1.805 0.02 rpy=0 0 0; parent main_field -> base_point
