Commit message: modify robot model, Lidar

File: sim/robot.urdf (robot description, URDF)
Before this commit: robot two_wheel_robot, 4 links, 3 joints
Links:
- link base_link: geometry collision box size=0.1 0.1 0.06; visual box size=0.1 0.1 0.06
- link left_wheel: geometry collision cylinder length=0.01 radius=0.03; visual cylinder length=0.01 radius=0.03
- link lidar_link: geometry collision box size=0.01 0.01 0.01; visual box size=0.01 0.01 0.01
- link right_wheel: geometry collision cylinder length=0.01 radius=0.03; visual cylinder length=0.01 radius=0.03
Joints:
- joint lidar_joint: origin xyz=0.05 0 0 rpy=0 0 0 -> xyz=0.055 0 0 rpy=0 0 0

Commit message: update

File: sim/robot.urdf (robot description, URDF)
Before this commit: robot two_wheel_robot, 4 links, 3 joints
Links:
- link base_link: geometry collision box size=0.1 0.1 0.059; visual box size=0.1 0.1 0.059
